File: electronics/project.sch (KiCad schematic (older format))
At the start: 9 parts

Commit message: W.I.P software
Parts:
- added C?: 22pF, symbol Device:C
Connections:
- wire segments 44 -> 45
Other:
- moved on the sheet: R?
Changed lines of the file:
@@
 Wire Wire Line
 	8050 3200 8600 3200
-Wire Wire Line
-	9500 4500 9700 4500
-Text GLabel 9700 4500 2    50   Input ~ 0
+Text GLabel 10150 4500 2    50   Input ~ 0
 3V3
 $Comp
 L Device:R R?
 U 1 1 5FF4B056
-P 10100 4600
-F 0 "R?" V 9893 4600 50  0000 C CNN
-F 1 "100k" V 9984 4600 50  0000 C CNN
-F 2 "" V 10030 4600 50  0001 C CNN
-F 3 "~" H 10100 4600 50  0001 C CNN
-	1    10100 4600
-	0    1    1    0
+P 10100 4750
+F 0 "R?" V 9893 4750 50  0000 C CNN
+F 1 "100k" V 9984 4750 50  0000 C CNN
+F 2 "" V 10030 4750 50  0001 C CNN
+F 3 "~" H 10100 4750 50  0001 C CNN
+	1    10100 4750
+	-1   0    0    1
 $EndComp
-Wire Wire Line
-	9950 4600 9500 4600
-Text GLabel 10250 4600 2    50   Input ~ 0
+Text GLabel 10100 4900 3    50   Input ~ 0
 GND
 $Comp
@@
 Text Notes 7400 7500 0    50   ~ 0
 Rocket1 flight controller\n
+$Comp
+L Device:C C?
+U 1 1 5FF15A10
+P 10000 4350
+F 0 "C?" V 9748 4350 50  0000 C CNN
+F 1 "22pF" V 9839 4350 50  0000 C CNN
+F 2 "" H 10038 4200 50  0001 C CNN
+F 3 "~" H 10000 4350 50  0001 C CNN
+	1    10000 4350
+	1    0    0    -1
+$EndComp
+Wire Wire Line
+	9500 4600 10100 4600
+Wire Wire Line
+	9500 4500 10000 4500
+Connection ~ 10000 4500
+Wire Wire Line
+	10000 4500 10150 4500
 $EndSCHEMATC

Commit message: first draft of controller and gateway
Parts:
- added R? (x2): 500k, symbol Device:R
- C?: value 22pF -> 10nF
Connections:
- net labels added: bat_read
- wire segments 45 -> 51
Changed lines of the file:
@@
 P 10000 4350
 F 0 "C?" V 9748 4350 50  0000 C CNN
-F 1 "22pF" V 9839 4350 50  0000 C CNN
+F 1 "10nF" V 9839 4350 50  0000 C CNN
 F 2 "" H 10038 4200 50  0001 C CNN
 F 3 "~" H 10000 4350 50  0001 C CNN
@@
 Wire Wire Line
 	10000 4500 10150 4500
+Wire Wire Line
+	6750 3500 6850 3500
+Wire Wire Line
+	6850 3500 6850 3600
+Wire Wire Line
+	6850 3600 7250 3600
+Text Label 7250 3600 2    50   ~ 0
+bat_read
+$Comp
+L Device:R R?
+U 1 1 5FF454D8
+P 2300 1600
+F 0 "R?" V 2507 1600 50  0000 C CNN
+F 1 "500k" V 2416 1600 50  0000 C CNN
+F 2 "" V 2230 1600 50  0001 C CNN
+F 3 "~" H 2300 1600 50  0001 C CNN
+	1    2300 1600
+	-1   0    0    1
+$EndComp
+$Comp
+L Device:R R?
+U 1 1 5FF468AF
+P 2300 2000
+F 0 "R?" V 2507 2000 50  0000 C CNN
+F 1 "500k" V 2416 2000 50  0000 C CNN
+F 2 "" V 2230 2000 50  0001 C CNN
+F 3 "~" H 2300 2000 50  0001 C CNN
+	1    2300 2000
+	-1   0    0    1
+$EndComp
+Wire Wire Line
+	2300 1850 2300 1800
+Text GLabel 2300 2150 3    50   Input ~ 0
+GND
+Wire Wire Line
+	2300 1800 2700 1800
+Connection ~ 2300 1800
+Wire Wire Line
+	2300 1800 2300 1750
+Text Label 2700 1800 2    50   ~ 0
+bat_read
 $EndSCHEMATC

Commit message: update protocol and schematics
Parts:
- C?: value 10nF -> 22pF
Connections:
- wire segments 51 -> 52
Changed lines of the file:
@@
 P 10000 4350
 F 0 "C?" V 9748 4350 50  0000 C CNN
-F 1 "10nF" V 9839 4350 50  0000 C CNN
+F 1 "22pF" V 9839 4350 50  0000 C CNN
 F 2 "" H 10038 4200 50  0001 C CNN
 F 3 "~" H 10000 4350 50  0001 C CNN
@@
 Text Label 2700 1800 2    50   ~ 0
 bat_read
+Text GLabel 10000 4200 1    50   Input ~ 0
+GND
+Wire Wire Line
+	4150 3200 4550 3200
+Text Label 4150 3200 0    50   ~ 0
+RF-RST
 $EndSCHEMATC

Commit message: new flight controller tested
Parts:
- removed R? (x2): 100k, symbol Device:R
- removed U?: Teensy4.0, symbol teensy:Teensy4.0
- removed U?: BMP280, symbol custom:BMP280
- removed U?: GY521, symbol custom:GY521
- removed U?: W25Q32JVDAIQ, symbol custom:W25Q32JVDAIQ
- added BZ1: Buzzer, custom:buzzer, symbol Device:Buzzer
- added D1: LED_RGBC, custom:LED_D5.0mm-4_RGB, symbol Device:LED_RGBC
- added J1: Conn_01x10, custom:01x10_header, symbol Connector_Generic:Conn_01x10
- added R3, R4: 330, Resistor_THT:R_Axial_DIN0207_L6.3mm_D2.5mm_P5.08mm_Vertical, symbol Device:R
- added R5: 1000, Resistor_THT:R_Axial_DIN0207_L6.3mm_D2.5mm_P5.08mm_Vertical, symbol Device:R
- added U1: teensy4, custom:teensy4, symbol custom:teensy4
- added U3: GY91, custom:GY91, symbol custom:GY91
- added U4: W25Q128JV, Package_SO:SOIC-8_5.275x5.275mm_P1.27mm, symbol custom:W25Q128JV
- BAT1: renamed from BAT; footprint (none) -> custom:terminal-small
- C1, C2: renamed from C?; footprint (none) -> Resistor_THT:R_Axial_DIN0207_L6.3mm_D2.5mm_P5.08mm_Vertical
- R1, R2: renamed from R?; value 500k -> 4.7k; footprint (none) -> Resistor_THT:R_Axial_DIN0207_L6.3mm_D2.5mm_P5.08mm_Vertical
- U2: renamed from U?; footprint (none) -> custom:Adafruit-RFM69
Connections:
- net labels added: BUZZ, EXT-CS, FLASH-HOLD, FLASH-WP, LED-B, LED-G, LED-R, RX1, TX1
- wire segments 52 -> 76
Other:
- moved on the sheet: C1
