File: electronics/v1/project.kicad_pcb (KiCad board)
At the start: 2 copper layers, 35.6 x 67.9 mm, 17 parts, among them J1 Conn_01x10, U1 Teensy 4.0, U2 RFM69HCW, U3 GY91, U4 W25Q128JV

Commit message: PCB mostly finished
Parts:
- R1, R2: value 500k -> 4.7k
- R3, R4: value R -> 330
- R5: value R -> 1000
- U1: value Teensy 4.0 -> teensy4
