File: electronics/main_v1/main_v1.kicad_pcb (KiCad board)
At the start: 4 copper layers, 100.3 x 100.3 mm, 139 parts, among them J1 JST_GH_6, J2 JST_XH_4, J3 JST_XH_4, J4 JST_GH_6, J5 JST_XH_4, J6 JST_GH_6, J7 JST_XH_4, J8 JST_XH_4, J9 Conn_Coaxial, Q1 DMG2301L, Q10 MMBT3904, Q11 MMBT3904, Q2 DMG2301L, Q3 PMN48XP, Q4 DMG2301L, Q5 DMG2301L, Q6 DMG2301L, Q7 DMG2301L, Q8 MMBT3904, Q9 PMN48XP, SW1 SW_DPST_x2, U1 Teensy4.1, U10 terminal-2, U11 BTN7030-1EPA, U12 BTN7030-1EPA, U13 BTN7030-1EPA, U14 BTN7030-1EPA, U15 NL17SZ17, U16 w25nxx, U17 SN65HVD230, U18 NL17SZ17, U19 NL17SZ17, U2 12v-engine, U20 NL17SZ17, U21 NL17SZ17, U23 terminal-2, U24 terminal-2, U25 BTN7030-1EPA, U26 BTN7030-1EPA, U27 12v-in, U28 7v-in, U29 L7805, U3 12v-out, U30 Si7021-A20, U31 ltc2992, U32 RFM98W-433S2, U33 GY91, U34 drotek_10dof, U35 drotek_10dof, U4 NL17SZ17, U5 NL17SZ17, U6 TXS0104EPWRG4, U7 terminal-2, U8 terminal-2, U9 terminal-2

Commit message: pre routing mini controller
Parts:
- removed D3: D_Schottky, Diode_SMD:D_0805_2012Metric_Pad1.15x1.40mm_HandSolder
- removed H3: Logo, custom:avatar
- removed Q1: DMG2301L, Package_TO_SOT_SMD:SOT-23
- removed R1: 1k, Resistor_SMD:R_0805_2012Metric_Pad1.20x1.40mm_HandSolder
- removed R18, R33, R37: 10k, Resistor_SMD:R_0805_2012Metric_Pad1.20x1.40mm_HandSolder
- removed R34: 60k, Resistor_SMD:R_0805_2012Metric_Pad1.20x1.40mm_HandSolder
- removed R38: 40k, Resistor_SMD:R_0805_2012Metric_Pad1.20x1.40mm_HandSolder
- removed U34: drotek_10dof, custom:drotek_10dof
- added C22: 100nf, Capacitor_SMD:C_0805_2012Metric_Pad1.18x1.45mm_HandSolder, B.Cu at (202.8, 82.5)
- added HS1: Heatsink_Pad, custom:d2pak_heatsink, B.Cu at (171.4, 135.9)
- added J10: JST_SH_4, Connector_JST:JST_SH_SM04B-SRSS-TB_1x04-1MP_P1.00mm_Horizontal, F.Cu at (237.5, 153.7)
- added JP3: Jumper, Connector_PinHeader_2.54mm:PinHeader_1x02_P2.54mm_Vertical, B.Cu at (230.5, 156.8)
- added JP4: Jumper_NO_Small, custom:R_1812_4532Metric_Pad1.30x3.40mm_HandSolder_no_silk, F.Cu at (158.1, 129.5)
- added U22: NL17SZ17, custom:SC-74-a, B.Cu at (209.6, 82.5)
- C21, Q6, R15, U20: moved to F.Cu
- D11: footprint Diode_SMD:D_0805_2012Metric_Pad1.15x1.40mm_HandSolder -> Diode_SMD:D_SOD-323_HandSoldering
- D13: value CUHS20S30 -> D_Schottky; footprint Diode_SMD:D_0805_2012Metric_Pad1.15x1.40mm_HandSolder -> Diode_SMD:D_SOD-323_HandSoldering
- J1: value JST_GH_6 -> JST_SH_4; footprint Connector_JST:JST_GH_BM06B-GHS-TBT_1x06-1MP_P1.25mm_Vertical -> Connector_JST:JST_SH_SM04B-SRSS-TB_1x04-1MP_P1.00mm_Horizontal
- R10: value 10k -> 4.7k
- R16: value 4.7k -> 1k; moved to F.Cu
- R41: value 4.7k -> 2k
- R7: value 4.7k -> 1k
- U29: moved to B.Cu
- U4: value NL17SZ17 -> TXS0104E; footprint custom:SC-74-a -> Package_SO:TSSOP-14_4.4x5mm_P0.65mm
- U6: value TXS0104EPWRG4 -> sparkfun_H3LIS331DL; footprint Package_SO:TSSOP-14_4.4x5mm_P0.65mm -> custom:sparkfun_H3LIS331DL
- moved U6 32.5 mm to (227.3, 101.6)
- moved U5 30.7 mm to (226.7, 126.4), turned to 0 degrees
- moved J4 26.7 mm to (237.5, 120.7)
- moved Q2 26.4 mm to (232.4, 125.1), turned to 90 degrees
- moved R3 26.1 mm to (231.1, 128.3), turned to 0 degrees
- moved C20 24.8 mm to (231.5, 153.0), turned to 0 degrees
- moved R16 19.9 mm to (177.9, 121.2), turned to 180 degrees
- moved R10 16.1 mm to (177.9, 123.2), turned to 180 degrees
- moved C21 15.7 mm to (230.5, 150.1)
- moved Q6 14.0 mm to (232.4, 138.4)
- moved J6 13.3 mm to (237.5, 134.0)
- moved J1 11.4 mm to (237.5, 145.4), turned to 90 degrees
- moved U4 10.1 mm to (229.9, 149.2), turned to 0 degrees
- moved R15 9.92 mm to (231.8, 134.3), turned to 270 degrees
- moved U20 8.82 mm to (228.0, 133.3), turned to 90 degrees
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Connections:
- C10 pad 2: 12V -> 12V_LIMIT
- C11 pad 2: 12V -> 12V_LIMIT
- C12 pad 2: 12V -> 12V_LIMIT
- C13 pad 2: 12V -> 12V_LIMIT
- C14 pad 2: 12V -> 12V_LIMIT
- C15 pad 2: 12V -> 12V_LIMIT
- C16 pad 1: Net-(C16-Pad1) -> 7V
- C20 pad 1: 5V -> GND
- C20 pad 2: GND -> 5V
- C9 pad 1: Net-(C9-Pad1) -> 5V
- D2 pad 3: Net-(C9-Pad1) -> 5V
- D2 pad 4: (no net) -> Net-(D2-Pad4)
- D9 pad 3: Net-(C9-Pad1) -> 5V
- J1 pad 2: Net-(J1-Pad2) -> 3V3
- J1 pad 3: Net-(J1-Pad3) -> /SDA0
- J1 pad 4: Net-(J1-Pad4) -> /SCL0
- J2 pad 1: GND -> Net-(J2-Pad1)
- J2 pad 2: Net-(J2-Pad2) -> GND
- J3 pad 1: GND -> 5V
- J3 pad 2: Net-(J2-Pad2) -> GND
- J3 pad 4: 5V -> Net-(J2-Pad4)
- J5 pad 4: (no net) -> 5V
- Q7 pad 3: Net-(J2-Pad4) -> Net-(J2-Pad1)
- Q9 pad 4: 12V -> 7V
- R16 pad 1: Net-(R16-Pad1) -> /UNSAFE_P_EN
- R16 pad 2: GND -> Net-(R16-Pad2)
- R2 pad 1: Net-(J2-Pad2) -> Net-(J2-Pad4)
- R2 pad 2: Net-(J2-Pad3) -> Net-(JP3-Pad2)
- R26 pad 2: 12V -> 7V
- R32 pad 2: Net-(C16-Pad1) -> 7V
- R7 pad 1: Net-(R16-Pad1) -> Net-(R16-Pad2)
- SW1 pad 1: /UNSAFE_P_EN -> GND
- SW1 pad 2: Net-(R16-Pad1) -> Net-(R16-Pad2)
- U1 pad 38: /EXTHV_RX -> (no net)
- U1 pad 39: /EXTHV_TX -> /RGB_TX
- U1 pad 45: /EXTHV_MOS -> (no net)
- U11 pad 15: 12V -> 12V_LIMIT
- U12 pad 15: 12V -> 12V_LIMIT
- U13 pad 15: 12V -> 12V_LIMIT
- U14 pad 15: 12V -> 12V_LIMIT
- U17 pad 7: Net-(J2-Pad2) -> Net-(J2-Pad4)
- U25 pad 15: 12V -> 12V_LIMIT
- U26 pad 15: 12V -> 12V_LIMIT
- U29 pad 1: Net-(C16-Pad1) -> 7V
- U31 pad 1: Net-(C16-Pad1) -> 7V
- U31 pad 12: GND -> (no net)
- U31 pad 14: Net-(R33-Pad2) -> (no net)
- U31 pad 3: Net-(R37-Pad1) -> (no net)
- U4 pad 1: (no net) -> 3V3
- U4 pad 2: /EXTHV_MOS -> (no net)
- U4 pad 3: GND -> (no net)
- U4 pad 4: Net-(R1-Pad1) -> /SDA0
- U4 pad 5: 5V -> /SCL0
- U6 pad 1: 3V3 -> (no net)
- U6 pad 2: /SDA0 -> (no net)
- U6 pad 3: /SCL0 -> (no net)
- U6 pad 4: /EXTHV_TX -> (no net)
- U6 pad 5: /EXTHV_RX -> /SCL2
- U6 pad 6: (no net) -> /SDA2
- U6 pad 7: GND -> 3V3
- U6 pad 8: 3V3 -> GND
Routing:
- net /RGB_TX: track 0.00 -> 86.1 mm
- net 12V: track 89.0 -> 23.7 mm
- net /EXTHV_MOS: track 62.0 -> 0.00 mm, vias 1 -> 0
- net 7V: track 0.00 -> 60.8 mm, vias 0 -> 9
- net 12V_LIMIT: track 0.00 -> 57.1 mm
- net /EXTHV_TX: track 45.6 -> 0.00 mm, vias 1 -> 0
- net /EXTHV_RX: track 45.4 -> 0.00 mm, vias 1 -> 0
- net 5V: track 232.7 -> 273.9 mm, vias 8 -> 7
- net /SDA0: track 180.9 -> 150.4 mm
- net Net-(R16-Pad2): track 0.00 -> 25.8 mm, vias 0 -> 1
- net Net-(C9-Pad1): track 24.4 -> 0.00 mm
- net Net-(C16-Pad1): track 22.5 -> 0.00 mm
- net Net-(J2-Pad2): track 21.4 -> 0.00 mm
- net /EXT_TX: track 78.2 -> 60.0 mm, vias 1 -> 0
- net /SCL0: track 168.0 -> 150.3 mm, vias 1 -> 3
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- added copper zone on In2.Cu, net GND
Other:
- outline, holes or cut-outs redrawn
- board text added: "CAN"
- board text added: "CAN always on"
- board text added: "Extra"
- board text added: "Extra1"
- board text added: "FPV"
- board text added: "GPS"
- board text added: "I2C 3V"
- board text added: "I2C 5V"
- board text added: "JLCJLCJLCJLC"
- board text added: "Telemetry"
- board text added: "V1.0 05-21"
- board text added: "liftoff"
- board text added: "never power up without antenna"
- board text added: "pyro off"
- board text removed: "Arm me!"
