File: electronics/main_v1/main_v1.sch (KiCad schematic (older format))
At the start: 139 parts, among them J1 JST_GH_6, J2 JST_XH_4, J3 JST_XH_4, J4 JST_GH_6, J5 JST_XH_4, J6 JST_GH_6, J7 JST_XH_4, J8 JST_XH_4, J9 Conn_Coaxial, Q1 DMG2301L, Q10 MMBT3904, Q11 MMBT3904, Q2 DMG2301L, Q3 PMN48XP, Q4 DMG2301L, Q5 DMG2301L, Q6 DMG2301L, Q7 DMG2301L, Q8 MMBT3904, Q9 PMN48XP, SW1 SW_DPST_x2, U1 Teensy4.1, U10 terminal-2, U11 BTN7030-1EPA, U12 BTN7030-1EPA, U13 BTN7030-1EPA, U14 BTN7030-1EPA, U15 NL17SZ17, U16 w25nxx, U17 SN65HVD230, U18 NL17SZ17, U19 NL17SZ17, U2 12v-engine, U20 NL17SZ17, U21 NL17SZ17, U23 terminal-2, U24 terminal-2, U25 BTN7030-1EPA, U26 BTN7030-1EPA, U27 12v-in, U28 7v-in, U29 L7805, U3 12v-out, U30 Si7021-A20, U31 ltc2992, U32 RFM98W-433S2, U33 GY91, U34 drotek_10dof, U35 drotek_10dof, U4 NL17SZ17, U5 NL17SZ17, U6 TXS0104EPWRG4, U7 terminal-2, U8 terminal-2, U9 terminal-2

Commit message: pre routing mini controller
Parts:
- removed D3: D_Schottky, Diode_SMD:D_0805_2012Metric_Pad1.15x1.40mm_HandSolder, symbol Device:D_Schottky
- removed H3: Logo, custom:avatar, symbol Mechanical:MountingHole
- removed J1: JST_GH_6, Connector_JST:JST_GH_BM06B-GHS-TBT_1x06-1MP_P1.25mm_Vertical, symbol Connector_Generic:Conn_01x06
- removed Q1: DMG2301L, Package_TO_SOT_SMD:SOT-23, symbol Transistor_FET:DMG2301L
- removed R1: 1k, Resistor_SMD:R_0805_2012Metric_Pad1.20x1.40mm_HandSolder, symbol Device:R
- removed R18, R33, R37: 10k, Resistor_SMD:R_0805_2012Metric_Pad1.20x1.40mm_HandSolder, symbol Device:R
- removed R34: 60k, Resistor_SMD:R_0805_2012Metric_Pad1.20x1.40mm_HandSolder, symbol Device:R
- removed R38: 40k, Resistor_SMD:R_0805_2012Metric_Pad1.20x1.40mm_HandSolder, symbol Device:R
- removed U34: drotek_10dof, custom:drotek_10dof, symbol custom:drotek_10dof
- removed U4: NL17SZ17, custom:SC-74-a, symbol custom:buffer
- removed U6: TXS0104EPWRG4, Package_SO:TSSOP-14_4.4x5mm_P0.65mm, symbol custom:TXS0104E
- added C22: 100n, Capacitor_SMD:C_0805_2012Metric_Pad1.18x1.45mm_HandSolder, symbol Device:C
- added HS1: Heatsink_Pad, custom:d2pak_heatsink, symbol Mechanical:Heatsink_Pad
- added J1, J10: JST_SH_4, Connector_JST:JST_SH_SM04B-SRSS-TB_1x04-1MP_P1.00mm_Horizontal, symbol Connector_Generic:Conn_01x04
- added JP3: Jumper, Connector_PinHeader_2.54mm:PinHeader_1x02_P2.54mm_Vertical, symbol Device:Jumper_NC_Small
- added JP4: Jumper_NO_Small, custom:R_1812_4532Metric_Pad1.30x3.40mm_HandSolder_no_silk, symbol Device:Jumper_NO_Small
- added U22: NL17SZ17, custom:SC-74-a, symbol custom:buffer
- added U4: TXS0104E, Package_SO:TSSOP-14_4.4x5mm_P0.65mm, symbol custom:TXS0104E
- added U6: sparkfun_H3LIS331DL, custom:sparkfun_H3LIS331DL, symbol custom:sparkfun_H3LIS331DL
- BZ1: mouser (none) -> 490-CX-0905C
- C1, C10, C11, C12, C13, C14, C15, C18, C19, C20, C21, C3, C4, C5, C6, C7, C8: mouser (none) -> 710-885012207072
- C16: value 330nF -> 330n; mouser (none) -> 80-C0805C334K3N
- C17: value 100nF -> 100n; mouser (none) -> 710-885012207072
- C2: value 100pF -> 100n; mouser (none) -> 710-885012207072
- C9: value 100nf -> 100n; mouser (none) -> 710-885012207072
- D1, D10, D12, D4, D6, D8: mouser (none) -> 621-SD15C-7
- D11: footprint Diode_SMD:D_0805_2012Metric_Pad1.15x1.40mm_HandSolder -> Diode_SMD:D_SOD-323_HandSoldering; mouser (none) -> 726-BAT60AE6327XT
- D13: value CUHS20S30 -> D_Schottky; footprint Diode_SMD:D_0805_2012Metric_Pad1.15x1.40mm_HandSolder -> Diode_SMD:D_SOD-323_HandSoldering; mouser (none) -> 726-BAT60AE6327XT
- D5: mouser (none) -> 710-150060AS75000
- D7: mouser (none) -> 710-150060YS75000
- J9: mouser (none) -> 712-CONSMA020.062-G
- Q10, Q11, Q8: mouser (none) -> 241-MMBT3904R200001
- Q2, Q4, Q5, Q6, Q7: mouser (none) -> 621-DMG2301L-7
- Q3, Q9: mouser (none) -> 771-PMN48XP,125
- R10: value 10k -> 4.7k; mouser (none) -> 652-CR0805FX-4701ELF
- R11, R12: value 400 -> 402; mouser (none) -> 603-RT0805FRE07402RL
- R13, R14, R15, R17, R25, R27, R3, R39, R4, R9: mouser (none) -> 667-ERJ-6ENF1001V
- R16, R7: value 4.7k -> 1k; mouser (none) -> 667-ERJ-6ENF1001V
- R19, R20, R21, R22, R23, R24, R28, R40, R5, R6, R8: mouser (none) -> 71-CRCW080510K0FKEAC
- R2: mouser (none) -> 652-CR0805FX-1200ELF
- R26, R29, R30, R35, R36: mouser (none) -> 652-CR0805FX-4701ELF
- R32: mouser 71-WSL2512R0250FEA -> WSL2512R0250FEB
- R41: value 4.7k -> 2k; mouser (none) -> 71-CRCW08052K00FKEAC
- U11, U12, U13, U14, U25, U26: mouser (none) -> 726-BTN70301EPAXUMA1
- U15, U18, U19, U20, U21, U5: mouser (none) -> 863-NL17SZ17DBVT1G
- U16: mouser (none) -> 454-W25N01GVSFIG
- U17: mouser (none) -> 595-SN65HVD231QDRQ1
- U29: mouser (none) -> 511-L7805ABD2T-TR
- U30: mouser (none) -> 634-SI7021-A20-IM
- U31: mouser (none) -> 584-LTC2992IMSPBF
- U32: mouser (none) -> :(
Connections:
- net 12V: now also JP4.1; no longer C10.2, C11.2, C12.2, C13.2, C14.2, C15.2, Q9.4 (S), R26.2, U11.15 (VS), U12.15 (VS), U13.15 (VS), U14.15 (VS), U25.15 (VS), U26.15 (VS)
- net 3V3: now also J1.2 (Pin_2), U4.1 (VCC_A), U4.8 (OE), U6.7 (3.3V)
- net 5V: now also C20.2, C9.1, D2.3 (VSS), D9.3 (VSS), J3.1 (Pin_1), J5.4 (Pin_4), C22.1, J10.2 (Pin_2), U22.5 (VCC), U4.14 (VCC_B); no longer C20.1, J3.4 (Pin_4)
- net Earth: now also C20.1, J2.2 (Pin_2), J3.2 (Pin_2), SW1.1 (A), C22.2, HS1.1, J1.1 (Pin_1), J10.1 (Pin_1), U22.3 (GND), U4.7 (GND), U6.8 (GND); no longer C20.2, J2.1 (Pin_1), J3.1 (Pin_1), R16.2, U31.12 (GND)
- net SCL0: now also J1.4 (Pin_4), U4.5 (A4)
- net SCL2: now also U6.5 (SCL)
- net SDA0: now also J1.3 (Pin_3), U4.4 (A3)
- net SDA2: now also U6.6 (SDA)
- net UNSAFE_P_EN: now also R16.1; no longer SW1.1 (A)
- net at R7.1, SW1.2 (B): now also R16.2; no longer R16.1
- net 7V: now reaches C16.1, R32.2, U29.1 (IN), U31.1 (sense_1-)
- net 7V: now also Q9.4 (S), R26.2
- net at R2.1, U17.7 (CANH): now also J2.4 (Pin_4), J3.4 (Pin_4); no longer J2.2 (Pin_2), J3.2 (Pin_2)
- net at J2.3 (Pin_3), J3.3 (Pin_3), U17.6 (CANL): now also JP3.1; no longer R2.2
- net at Q7.3 (D): now also J2.1 (Pin_1); no longer J2.4 (Pin_4)
- net EXTHV_MOS: no longer names the net of U1.45 (23_A9_CRX1_MCLK1)
- net EXTHV_RX: no longer names the net of U1.38 (16_A2_RX4_SCL1)
- net EXTHV_TX renamed RGB_TX
- net RGB_TX: now also U22.2 (IN)
- net RGB: no longer names the net of D2.4 (DIN)
- net RGB: now also U22.4 (OUT)
- new net: JP3.2, R2.2
- new net: J10.3 (Pin_3), U4.11 (B3)
- new net: J10.4 (Pin_4), U4.10 (B4)
- new net 12V_LIMIT: C10.2, C11.2, C12.2, C13.2, C14.2, C15.2, JP4.2, U11.15 (VS), U12.15 (VS), U13.15 (VS), U14.15 (VS), U25.15 (VS), U26.15 (VS)
- no-connect marks 7 -> 6
Other:
- note added: "3v3 qwiic"
- note added: "5V qwiic"
- note removed: "extraHV"
- moved on the sheet: D6, JP2, Q7, R17, R2, R24, R41, R7, U21
