File: electronics/v2/fc_v2.kicad_pcb (KiCad board)
At the start: 2 copper layers, 36.1 x 87.9 mm, 45 parts, among them J1 Conn_02x03_Counter_Clockwise, Q1 Q_NPN, SW1 SW_DPST_x2, U1 Teensy 4.0, U10 terminal-2, U11 BTN7030-1EPA, U12 BTN7030-1EPA, U13 BTN7030-1EPA, U14 BTN7030-1EPA, U2 RFM69HCW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

Commit message: fixes on PCB
Parts:
- added D1: D_Schottky, Diode_SMD:D_0805_2012Metric_Pad1.15x1.40mm_HandSolder, B.Cu at (131.7, 105.8)
- added H1: MountingHole, MountingHole:MountingHole_2.2mm_M2_ISO7380, F.Cu at (125.9, 63.8)
- added H2: MountingHole, MountingHole:MountingHole_2.2mm_M2_ISO7380, F.Cu at (153.0, 63.8)
- added H3: Logo, custom:avatar, F.Cu at (140.3, 102.6)
- added H4: MountingHole, MountingHole:MountingHole_2.2mm_M2_ISO7380, F.Cu at (125.9, 155.2)
- added H5: MountingHole, MountingHole:MountingHole_2.2mm_M2_ISO7380, F.Cu at (153.0, 155.2)
- added R6: 10k, Resistor_SMD:R_0805_2012Metric_Pad1.20x1.40mm_HandSolder, B.Cu at (131.1, 137.1)
- added R7: 4.7k, Resistor_SMD:R_0805_2012Metric_Pad1.20x1.40mm_HandSolder, F.Cu at (146.2, 102.2)
- added R9: 2k, Resistor_SMD:R_0805_2012Metric_Pad1.20x1.40mm_HandSolder, B.Cu at (127.5, 139.6)
- C2: value 22pF -> 100pF
- R1, R2: moved to B.Cu
- R14, R15: value 330 -> 700
- R16: value 10k -> 4.7k
- U1: value Teensy 4.0 -> teensy4
- U4: footprint Package_SO:SOIC-8_7.5x5.85mm_P1.27mm -> Package_SO:SOIC-8_5.275x5.275mm_P1.27mm
- U5: footprint Connector_AMASS:AMASS_XT30U-F_1x02_P5.0mm_Vertical -> Connector_AMASS:AMASS_XT30U-M_1x02_P5.0mm_Vertical
- moved Q1 6.69 mm to (130.9, 142.4), turned to 270 degrees
- moved D3 3.90 mm to (127.9, 105.4), turned to 0 degrees
- moved R1 2.43 mm to (143.4, 129.4), turned to 180 degrees
- moved C2 2.30 mm to (127.8, 86.1)
- moved C3 1.85 mm to (145.3, 110.2), turned to 0 degrees
- moved U5 1.27 mm to (151.8, 106.7)
- moved R2 0.51 mm to (143.8, 132.6)
- moved C7 0.23 mm to (147.8, 77.7)
Connections:
- C4 pad 1: 5V -> Net-(C4-Pad1)
- Q1 pad 1: /BUZZ -> Net-(Q1-Pad1)
- R16 pad 1: /P-EN -> Net-(R16-Pad1)
- SW1 pad 2: /P-EN -> Net-(R16-Pad1)
- U4 pad 3: GND -> 3V3
- U4 pad 7: GND -> 3V3
- U6 pad 3: 5V -> Net-(C4-Pad1)
Routing:
- net 12V: track 74.8 -> 143.2 mm, vias 2 -> 3
- net GND: track 245.5 -> 220.1 mm, vias 28 -> 50
- net Net-(R16-Pad1): track 0.00 -> 9.83 mm
- net 3V3: track 94.7 -> 104.2 mm
- net /BUZZ: track 7.16 -> 14.6 mm
- net /UNSAFE-P-EN: track 75.1 -> 68.1 mm
- net Net-(C4-Pad1): track 0.00 -> 5.81 mm
- net 5V: track 92.1 -> 86.3 mm
- net Net-(D2-Pad3): track 6.40 -> 2.60 mm
- net /RF-RST: track 70.0 -> 66.6 mm
- net Net-(Q1-Pad1): track 0.00 -> 2.81 mm
- net Net-(BZ1-Pad2): track 2.18 -> 4.27 mm
- net /FLASH-CS: track 94.5 -> 92.7 mm
- net /SCK: track 37.4 -> 39.1 mm
- net /MOSI: track 53.8 -> 55.6 mm
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- added copper zone on F.Cu, net 12V
Other:
- board size 36.1 x 87.9 mm -> 36.1 x 96.8 mm
- board text added: "21-5"
- board text added: "3V"
- board text added: "Arm me!"
- board text added: "GND"
- board text added: "JLCJLCJLCJLC"
- board text added: "RX"
- board text added: "SCL"
- board text added: "SDA"
- board text added: "TX"
- board text added: "V1.0"
- board text removed: "Arm me!!"

Commit message: fix P-EN
Parts:
- removed D13: ARMED, LED_SMD:LED_0805_2012Metric_Pad1.15x1.40mm_HandSolder
- removed D14: SAFE, LED_SMD:LED_0805_2012Metric_Pad1.15x1.40mm_HandSolder
- removed R14, R15: 700, Resistor_SMD:R_0805_2012Metric_Pad1.20x1.40mm_HandSolder
- added D5: ARMED, LED_SMD:LED_0805_2012Metric_Pad1.15x1.40mm_HandSolder, F.Cu at (136.8, 105.8)
- added D7: SAFE, LED_SMD:LED_0805_2012Metric_Pad1.15x1.40mm_HandSolder, F.Cu at (131.6, 105.8)
- added G***: LOGO, custom:aesir_square, B.Cu at (130.4, 71.9)
- added R10: 10k, Resistor_SMD:R_0805_2012Metric_Pad1.20x1.40mm_HandSolder, B.Cu at (149.4, 132.6)
- added R11: 400, Resistor_SMD:R_0805_2012Metric_Pad1.20x1.40mm_HandSolder, F.Cu at (132.5, 109.9)
- added R12: 400, Resistor_SMD:R_0805_2012Metric_Pad1.20x1.40mm_HandSolder, F.Cu at (135.9, 109.0)
- added U15: buffer, custom:SC-74-a, F.Cu at (136.1, 112.1)
- H3: moved to B.Cu
- R16: value 4.7k -> 10k
- moved H3 21.5 mm to (127.3, 119.6), turned to 180 degrees
Routing:
- net GND: track 220.1 -> 205.7 mm, vias 50 -> 51
- net Net-(D7-Pad1): track 0.00 -> 7.06 mm
- net 3V3: track 104.2 -> 111.1 mm, vias 2 -> 4
- net Net-(D5-Pad1): track 0.00 -> 6.02 mm
- net Net-(D5-Pad2): track 0.00 -> 4.33 mm
- net Net-(D13-Pad1): track 2.06 -> 0.00 mm
- net Net-(D14-Pad2): track 2.04 -> 0.00 mm
- net /UNSAFE-P-EN: track 68.1 -> 67.1 mm
Other:
- board text added: "Safe|Armed"
- board text removed: "Armed | Safe"

Commit message: main fc traces done
Parts:
- removed G***: LOGO, custom:aesir_square
- added C1: 100nF, Capacitor_SMD:C_0805_2012Metric_Pad1.18x1.45mm_HandSolder, B.Cu at (146.4, 149.6)
- added C9: C, Capacitor_SMD:C_0805_2012Metric_Pad1.18x1.45mm_HandSolder, B.Cu at (123.7, 105.4)
- added D11: D_Schottky, Diode_SMD:D_0805_2012Metric_Pad1.15x1.40mm_HandSolder, B.Cu at (127.9, 107.4)
- added D9: D_Schottky, Diode_SMD:D_0805_2012Metric_Pad1.15x1.40mm_HandSolder, B.Cu at (125.3, 136.0)
- added H6: Aesir, custom:aesir, B.Cu at (129.2, 69.7)
- added J2: JST_XH_4, Connector_JST:JST_XH_B4B-XH-A_1x04_P2.50mm_Vertical, B.Cu at (126.4, 131.7)
- added R13: 120, Resistor_SMD:R_0805_2012Metric_Pad1.20x1.40mm_HandSolder, B.Cu at (150.5, 142.5)
- added U16: w25nxx, Package_SO:SOIC-16W_7.5x10.3mm_P1.27mm, B.Cu at (128.1, 79.1)
- BZ1: footprint custom:buzzer -> custom:CX-0905C
- J1: value Conn_02x03_Counter_Clockwise -> Conn_02x03_Odd_Even
- Q1: value Q_NPN -> MMBT3904
- R16: value 10k -> 4.7k
- R9: value 2k -> 400
- U15: value buffer -> NL17SZ17
- U4: value W25Q128JV -> SN65HVD230; footprint Package_SO:SOIC-8_5.275x5.275mm_P1.27mm -> Package_SO:SOIC-8_3.9x4.9mm_P1.27mm
- moved U4 71.5 mm to (150.6, 148.1), turned to 90 degrees
- moved H3 29.3 mm to (130.6, 148.7)
- moved R5 9.27 mm to (125.1, 88.0)
- moved BZ1 3.96 mm to (129.7, 144.8)
- moved C2 3.01 mm to (130.4, 87.5), turned to 270 degrees
- moved D4 1.29 mm to (144.0, 149.6)
- moved R16 1.27 mm to (150.5, 103.4)
- moved SW1 0.51 mm to (151.4, 97.5)
- moved R4 0.40 mm to (131.4, 128.4)
- moved R3 0.40 mm to (131.4, 125.9)
- moved J1 0.13 mm to (125.1, 109.3)
Connections:
- net /BAT-READ renamed /BAT_READ
- net /EXT-RX renamed /EXT_RX
- net /EXT-TX renamed /EXT_TX
- net /P-EN renamed /P_EN
- net /P-IN-1 renamed /P_IN_1
- net /P-IN-2 renamed /P_IN_2
- net /P-IN-3 renamed /P_IN_3
- net /P-IN-4 renamed /P_IN_4
- net /RF-CS renamed /RF_CS
- net /RF-G0 renamed /RF_G0
- net /RF-RST renamed /RF_RST
- net /UNSAFE-P-EN renamed /UNSAFE_P_EN
- J1 pad 2: 3V3 -> Net-(D11-Pad1)
- R5 pad 2: /FLASH-CS -> /FLASH_CS
- U1 pad 12: /FLASH-CS -> /FLASH_CS
- U1 pad 2: (no net) -> /CAN_RX
- U1 pad 3: (no net) -> /CAN_TX
- U4 pad 1: /FLASH-CS -> /CAN_TX
- U4 pad 2: /MISO -> GND
- U4 pad 4: GND -> /CAN_RX
- U4 pad 5: /MOSI -> (no net)
- U4 pad 6: /SCK -> Net-(J2-Pad3)
- U4 pad 7: 3V3 -> Net-(J2-Pad2)
- U4 pad 8: 3V3 -> GND
Routing:
- net /FLASH_CS: track 0.00 -> 105.7 mm, vias 0 -> 2
- net /FLASH-CS: track 92.7 -> 0.00 mm
- net GND: track 205.7 -> 124.9 mm, vias 51 -> 55
- net 12V: track 143.2 -> 191.8 mm
- net Net-(J2-Pad2): track 0.00 -> 35.7 mm, vias 0 -> 1
- net Net-(J2-Pad3): track 0.00 -> 34.4 mm, vias 0 -> 1
- net /SCK: track 39.1 -> 58.5 mm
- net /MOSI: track 55.6 -> 68.0 mm
- net /MISO: track 64.3 -> 54.1 mm
- net /CAN_TX: track 0.00 -> 7.84 mm
- net /CAN_RX: track 0.00 -> 7.61 mm
- net Net-(D9-Pad2): track 0.00 -> 4.32 mm
- net 5V: track 86.3 -> 83.7 mm, vias 3 -> 2
- net Net-(BZ1-Pad2): track 4.27 -> 1.93 mm
- net Net-(C9-Pad1): track 2.60 -> 4.88 mm
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Other:
- board text added: "5V"
- board text removed: "3V"

Commit message: pre routing mini controller
Parts:
- removed D3: D_Schottky, Diode_SMD:D_0805_2012Metric_Pad1.15x1.40mm_HandSolder
- removed R16: 4.7k, Resistor_SMD:R_0805_2012Metric_Pad1.20x1.40mm_HandSolder
- added JP1: Jumper_NC_Small, Connector_PinHeader_2.54mm:PinHeader_1x02_P2.54mm_Vertical, B.Cu at (146.7, 139.7)
- added JP2: Jumper, Connector_JST:JST_XH_B2B-XH-A_1x02_P2.50mm_Vertical, B.Cu at (124.5, 148.0)
- added JP3: Jumper_NO_Small, custom:R_1812_4532Metric_Pad1.30x3.40mm_HandSolder_no_silk, B.Cu at (148.3, 96.8)
- added R14: 1k, Resistor_SMD:R_0805_2012Metric_Pad1.20x1.40mm_HandSolder, F.Cu at (154.4, 101.7)
- added R15: 2k, Resistor_SMD:R_0805_2012Metric_Pad1.20x1.40mm_HandSolder, F.Cu at (135.9, 148.9)
- added U17: NL17SZ17, custom:SC-74-a, B.Cu at (124.5, 99.7)
- C1: value 100nF -> 100n
- C2: value 100pF -> 100p
- C3: value 20uF -> 20u
- C4: value 10uF -> 10u
- C9: value C -> 100n
- D1, D11, D4, D9: footprint Diode_SMD:D_0805_2012Metric_Pad1.15x1.40mm_HandSolder -> Diode_SMD:D_SOD-323_HandSoldering
- H1, H2, H4, H5: value MountingHole -> MountingHole_Pad; footprint MountingHole:MountingHole_2.2mm_M2_ISO7380 -> MountingHole:MountingHole_2.2mm_M2_Pad_Via
- R1: value 6k -> 6.04k
- R10: value 10k -> 4.7k
- R7: value 4.7k -> 1k
- R9: value 400 -> 1k
- moved H1 95.6 mm to (152.9, 155.4)
- moved H5 91.7 mm to (152.9, 63.5)
- moved H2 27.1 mm to (126.0, 63.5)
- moved D9 16.7 mm to (124.0, 119.4)
- moved R13 3.81 mm to (150.4, 138.7)
- moved H3 3.61 mm to (134.1, 149.4)
- moved SW1 0.46 mm to (151.1, 97.2)
- moved H4 0.28 mm to (126.0, 155.4)
- moved D4 0.13 mm to (144.1, 149.6)
Connections:
- C10 pad 2: 12V -> 12V_LIMIT
- C12 pad 2: 12V -> 12V_LIMIT
- C9 pad 1: Net-(C9-Pad1) -> 5V
- D2 pad 3: Net-(C9-Pad1) -> 5V
- D2 pad 4: RGB -> Net-(D2-Pad4)
- H1 pad 1: (no net) -> GND
- H2 pad 1: (no net) -> GND
- H4 pad 1: (no net) -> GND
- H5 pad 1: (no net) -> GND
- J2 pad 1: Net-(D9-Pad2) -> Net-(J2-Pad1)
- J2 pad 3: Net-(J2-Pad3) -> GND
- J2 pad 4: GND -> Net-(D9-Pad2)
- R13 pad 1: Net-(J2-Pad2) -> Net-(J2-Pad1)
- R13 pad 2: Net-(J2-Pad3) -> Net-(JP1-Pad1)
- SW1 pad 1: /UNSAFE_P_EN -> GND
- U1 pad 27: (no net) -> /RGB_TX
- U1 pad 29: (no net) -> /LIFTOFF
- U1 pad 4: RGB -> (no net)
- U11 pad 15: 12V -> 12V_LIMIT
- U12 pad 15: 12V -> 12V_LIMIT
- U13 pad 15: 12V -> 12V_LIMIT
- U14 pad 15: 12V -> 12V_LIMIT
- U4 pad 6: Net-(J2-Pad3) -> Net-(J2-Pad2)
- U4 pad 7: Net-(J2-Pad2) -> Net-(J2-Pad1)
Routing:
- net 12V: track 191.8 -> 43.5 mm
- net 12V_LIMIT: track 0.00 -> 143.8 mm
- net RGB: track 60.6 -> 0.00 mm
- net /RGB_TX: track 0.00 -> 44.9 mm, vias 0 -> 1
- net Net-(J2-Pad1): track 0.00 -> 34.9 mm
- net Net-(J2-Pad3): track 34.4 -> 0.00 mm, vias 1 -> 0
- net /LIFTOFF: track 0.00 -> 24.5 mm
- net 3V3: track 112.6 -> 130.8 mm, vias 9 -> 8
- net /UNSAFE_P_EN: track 67.1 -> 60.2 mm
- net /P_EN: track 46.2 -> 40.7 mm
- net Net-(D2-Pad4): track 0.00 -> 5.23 mm
- net Net-(C9-Pad1): track 4.88 -> 0.00 mm
- net Net-(JP1-Pad1): track 0.00 -> 2.48 mm
- net Net-(D9-Pad2): track 4.32 -> 5.39 mm
- net 5V: track 83.7 -> 82.7 mm, vias 2 -> 1
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- added copper zone on F.Cu, net 12V_LIMIT
- removed copper zone on F.Cu, net 12V
Other:
- board size 36.1 x 96.8 mm -> 36.1 x 97 mm
- board text added: "pyro off"
- board text removed: "Arm me!"
