File: electronics/mini_controller/mini_controller.sch (KiCad schematic (older format))
At the start: 50 parts, among them J1 Conn_01x04, J2 Conn_01x04, J3 sma, J4 Conn_01x04, Q1 MMBT3904, SW1 chs-01a, U1 JST-RCY, U10 SKY65723-81, U11 SBE807, U12 ADXL343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

Commit message: pre U.FL version
Parts:
- removed C4: 2.2u, Capacitor_SMD:C_0603_1608Metric_Pad1.08x0.95mm_HandSolder, symbol Device:C_Small
- removed R9: 10k, Resistor_SMD:R_0603_1608Metric_Pad0.98x0.95mm_HandSolder, symbol Device:R_Small
- removed U11: SBE807, custom:SC-74-a, symbol custom:SBE807
- removed U3: AP2205-33W5, Package_TO_SOT_SMD:SOT-23-5_HandSoldering, symbol custom:AP2205-33W5
- added D1, D3: ZLLS350TA, Diode_SMD:D_SOD-523, symbol Device:D_Schottky_Small
- added J5: SWD port, Connector_PinHeader_1.27mm:PinHeader_1x04_P1.27mm_Vertical, symbol Connector_Generic:Conn_01x04
- added U3: NCV51460, Package_TO_SOT_SMD:SOT-23, symbol Regulator_Linear:APE8865NR-21-HF-3
- C1: value 1u -> 0.1u
- J1: value Conn_01x04 -> terminal 1
- J2: value Conn_01x04 -> terminal 2
Connections:
- net 3V3: now also C6.1, R11.1, R12.2, U10.1 (VCC), U10.2 (VEN), U12.1 (Vdd_I/O), U12.6 (Vs), U12.7 (~CS), J5.4 (Pin_4)
- net 3V3_BAK: now also U3.2 (VO)
- net BAT_SENSE: now also U8.6 (PC2)
- net BUZZER: no longer U8.13 (PA0)
- net GND: now also U12.12 (SDO/ADDR), U12.2 (GND), U12.4 (GND), U12.5 (GND), J5.1 (Pin_1), U3.3 (GND); no longer R11.1, R12.2
- net PYRO_1_EN: now also U8.25 (PB1_IO_INT2)
- net PYRO_2_EN: now also U8.24 (PB0_IO_INT1)
- net PYRO_3_EN: now also U8.7 (PC3)
- net PYRO_4_EN: now also U8.13 (PA0)
- net SCL3: now also U12.14 (SCL/SCLK); no longer U12.7 (~CS)
- net SDA3: now also U12.13 (SDA/SDI/SDIO); no longer U12.14 (SCL/SCLK)
- net SWCLK: now also J5.2 (Pin_2)
- net SWDIO: now also J5.3 (Pin_3)
- net at F1.1, U1.2 (+): now also C1.2, D1.2 (A), D3.2 (A), U3.1 (VI)
- net at C2.2, R1.1, U2.8 (VCC): now also D3.1 (K); no longer C1.2
- net at U4.13 (LNA_EN): no longer U10.2 (VEN)
- net at R7.1: now also D1.1 (K)
- now unconnected: U4.14 (VCC_RF)
Other:
- note added: "datasheet wants a resistor but it \nworks without, no space for it"
- note added: "no cap according to datasheet\nbuilt in reverse voltage\n"
- note removed: "GPS"
- moved on the sheet: C2, C3, F1, R1, R7, R8, U1, U12, U2, j1
