File: electronics/mini_controller/mini_controller.kicad_pcb (KiCad board)
At the start: 4 copper layers, 13.2 x 60.6 mm, 50 parts, among them J1 Conn_01x04, J2 Conn_01x04, J3 sma, J4 Conn_01x04, Q1 MMBT3904, SW1 chs-01a, U1 JST-RCY, U10 SKY65723-81, U11 SBE807, U12 ADXL343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

Commit message: pre U.FL version
Parts:
- removed C4: 2.2u, Capacitor_SMD:C_0603_1608Metric_Pad1.08x0.95mm_HandSolder
- removed R9: 10k, Resistor_SMD:R_0603_1608Metric_Pad0.98x0.95mm_HandSolder
- removed U11: SBE807, custom:SC-74-a
- added D1: ZLLS350TA, Diode_SMD:D_SOD-523, B.Cu at (135.4, 92.5)
- added D3: ZLLS350TA, Diode_SMD:D_SOD-523, B.Cu at (127.4, 110.7)
- added J5: SWD port, Connector_PinHeader_1.27mm:PinHeader_1x04_P1.27mm_Vertical, F.Cu at (124.7, 63.8)
- C1: value 1u -> 0.1u
- J1: value Conn_01x04 -> terminal 1
- J2: value Conn_01x04 -> terminal 2
- U3: value AP2205-33W5 -> NCV51460; footprint Package_TO_SOT_SMD:SOT-23-5_HandSoldering -> Package_TO_SOT_SMD:SOT-23
- moved R7 18.9 mm to (136.9, 92.4)
- moved R8 12.2 mm to (135.4, 89.1), turned to 90 degrees
- moved C1 6.65 mm to (135.7, 101.2), turned to 180 degrees
- moved R5 5.29 mm to (132.6, 69.5), turned to 180 degrees
- moved R6 4.09 mm to (127.9, 69.5), turned to 0 degrees
- moved R12 3.79 mm to (136.9, 89.1)
- moved U7 1.55 mm to (126.9, 103.6)
- moved C6 1.44 mm to (131.9, 104.9), turned to 0 degrees
- moved U1 0.77 mm to (136.0, 103.8)
- moved BZ1 0.50 mm to (127.6, 79.7), turned to 270 degrees
- moved R16 0.38 mm to (133.9, 110.8)
- moved U12 0.36 mm to (127.0, 86.0)
- moved U10 0.34 mm to (131.1, 103.0), turned to 270 degrees
- moved U4 0.28 mm to (129.3, 90.2), turned to 270 degrees
- moved U3 0.25 mm to (134.7, 98.5), turned to 270 degrees
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Connections:
- C2 pad 2: Net-(C1-Pad2) -> Net-(C2-Pad2)
- C6 pad 1: Net-(C6-Pad1) -> /3V3
- F1 pad 1: Net-(F1-Pad1) -> Net-(C1-Pad2)
- R1 pad 1: Net-(C1-Pad2) -> Net-(C2-Pad2)
- R11 pad 1: GND -> /3V3
- R12 pad 2: GND -> /3V3
- U1 pad 2: Net-(F1-Pad1) -> Net-(C1-Pad2)
- U10 pad 1: Net-(C6-Pad1) -> /3V3
- U10 pad 2: Net-(U10-Pad2) -> /3V3
- U12 pad 1: (no net) -> /3V3
- U12 pad 12: (no net) -> GND
- U12 pad 13: (no net) -> /SDA3
- U12 pad 14: /SDA3 -> /SCL3
- U12 pad 2: Net-(U12-Pad2) -> GND
- U12 pad 4: Net-(U12-Pad2) -> GND
- U12 pad 5: Net-(U12-Pad2) -> GND
- U12 pad 6: (no net) -> /3V3
- U12 pad 7: /SCL3 -> /3V3
- U2 pad 8: Net-(C1-Pad2) -> Net-(C2-Pad2)
- U3 pad 2: GND -> /3V3_BAK
- U3 pad 3: Net-(C1-Pad2) -> GND
- U4 pad 13: Net-(U10-Pad2) -> (no net)
- U4 pad 14: Net-(C6-Pad1) -> (no net)
- U8 pad 13: /BUZZER -> /PYRO_4_EN
- U8 pad 24: (no net) -> /PYRO_2_EN
- U8 pad 25: (no net) -> /PYRO_1_EN
- U8 pad 50: (no net) -> /SWDIO
- U8 pad 51: (no net) -> /SWCLK
- U8 pad 6: (no net) -> /BAT_SENSE
- U8 pad 7: (no net) -> /PYRO_3_EN
Routing:
- net /3V3: track 0.00 -> 114.0 mm, vias 0 -> 2
- net Net-(R1-Pad2): track 0.00 -> 68.9 mm, vias 0 -> 1
- net GND: track 0.00 -> 64.3 mm, vias 0 -> 19
- net /PYRO_2_EN: track 0.00 -> 58.6 mm, vias 0 -> 3
- net /PYRO_3_EN: track 0.00 -> 55.8 mm, vias 0 -> 4
- net /PYRO_1_EN: track 0.00 -> 53.9 mm, vias 0 -> 3
- net /LED_G: track 0.00 -> 46.4 mm, vias 0 -> 2
- net /PYRO_4_EN: track 0.00 -> 45.7 mm, vias 0 -> 3
- net /LED_R: track 0.00 -> 43.3 mm, vias 0 -> 2
- net /LED_B: track 0.00 -> 42.1 mm, vias 0 -> 2
- net /FLASH_CS: track 0.00 -> 41.7 mm, vias 0 -> 2
- net /FLASH_MISO: track 0.00 -> 41.4 mm, vias 0 -> 2
- net /V_BAT: track 0.00 -> 41.3 mm
- net /FLASH_MOSI: track 0.00 -> 35.7 mm, vias 0 -> 2
- net /FLASH_SCK: track 0.00 -> 32.5 mm, vias 0 -> 2
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
Commit message: mini controller finished
Parts:
- moved R8 13.1 mm to (125.9, 98.2), turned to 180 degrees
- moved R7 9.36 mm to (129.5, 98.2), turned to 180 degrees
- moved D1 6.36 mm to (132.7, 98.2), turned to 0 degrees
- moved U3 1.02 mm to (135.8, 98.5)
- moved C1 0.57 mm to (135.7, 101.8)
Routing:
- net Net-(R1-Pad2): track 68.9 -> 4.31 mm, vias 1 -> 0
- net /3V3: track 114.0 -> 127.7 mm
- net /BAT_SENSE: track 0.05 -> 7.21 mm, vias 0 -> 1
- net GND: track 64.3 -> 58.8 mm, vias 19 -> 17
- net Net-(C1-Pad2): track 30.6 -> 27.6 mm
- net /3V3_BAK: track 14.6 -> 12.1 mm
- net Net-(D1-Pad1): track 2.43 -> 3.98 mm
