File: electronics/mini_controller2/mini_controller.sch (KiCad schematic (older format))
At the start: 50 parts, among them J1 terminal 1, J2 terminal 2, J3 sma, J4 Conn_01x04, J5 SWD port, Q1 MMBT3904, SW1 chs-01a, U1 JST-RCY, U10 SKY65723-81, U12 ADXL343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

Commit message: mini controller finished
Parts:
- removed J3: sma, Connector_Coaxial:SMA_Molex_73251-2120_EdgeMount_Horizontal, symbol Connector:Conn_Coaxial_Power
- removed J5: SWD port, Connector_PinHeader_1.27mm:PinHeader_1x04_P1.27mm_Vertical, symbol Connector_Generic:Conn_01x04
- added AE2: ANT-868-PW-LP, custom:ANT-868-PW-LP, symbol Device:Antenna
- added C4: 0.1u, Capacitor_SMD:C_0603_1608Metric_Pad1.08x0.95mm_HandSolder, symbol Device:C_Small
- added J3: GND, custom:just_a_pad, symbol Connector_Generic:Conn_01x01
- added J5: 3V3, custom:just_a_pad, symbol Connector_Generic:Conn_01x01
- added J6: SWDIO, custom:just_a_pad, symbol Connector_Generic:Conn_01x01
- added J7: SWCLK, custom:just_a_pad, symbol Connector_Generic:Conn_01x01
- AE1: value SGGP.12A -> U.FL; footprint Connector_Coaxial:U.FL_Molex_MCRF_73412-0110_Vertical -> Connector_Coaxial:U.FL_Hirose_U.FL-R-SMT-1_Vertical
- U12: value ADXL343 -> ADXL375
- j1: footprint Connector_PinHeader_2.54mm:PinHeader_1x02_P2.54mm_Vertical_SMD_Pin1Left -> custom:PinHeader_1x02_P2.54mm_Vertical_SMD
Connections:
- net 3V3: now also J5.1 (Pin_1)
- net 3v3: now also C4.1
- net GND: now also C4.2, J3.1 (Pin_1)
- net LED_B: now also U8.28 (PC8); no longer U8.26 (PC6)
- net LED_G: now also U8.26 (PC6); no longer U8.28 (PC8)
- net LED_R: now also R3.1; no longer R3.2
- net SWCLK: now also J7.1 (Pin_1)
- net SWDIO: now also J6.1 (Pin_1)
- net at U8.33 (RF_ANT): now also AE2.1 (A)
- net at D2.2 (RA): now also R3.2; no longer R3.1
Other:
- note removed: "UFL VERSION"
Changed lines of the file:
@@
 F 0 "j1" H 1500 2200 50  0000 L CNN
 F 1 "power" H 1500 2150 50  0001 L CNN
-F 2 "Connector_PinHeader_2.54mm:PinHeader_1x02_P2.54mm_Vertical_SMD_Pin1Left" H 1600 2350 50  0001 C CNN
+F 2 "custom:PinHeader_1x02_P2.54mm_Vertical_SMD" H 1600 2350 50  0001 C CNN
 F 3 "~" H 1600 2350 50  0001 C CNN
 	1    1600 2350
 	1    0    0    -1
 $EndComp
-$Comp
-L Connector:Conn_Coaxial_Power J3
-U 1 1 611B0EF4
-P 7450 4000
-F 0 "J3" V 7750 3900 50  0000 C CNN
-F 1 "sma" V 7650 3900 50  0000 C CNN
-F 2 "Connector_Coaxial:SMA_Molex_73251-2120_EdgeMount_Horizontal" H 7450 3950 50  0001 C CNN
-F 3 "~" H 7450 3950 50  0001 C CNN
-	1    7450 4000
-	0    -1   -1   0
-$EndComp
-Wire Wire Line
-	7350 4000 7000 4000
 Wire Wire Line
 	7000 3900 7050 3900
 Wire Wire Line
-	7050 3900 7050 3850
-Wire Wire Line
 	7050 3800 7000 3800
-Connection ~ 7050 3850
-Wire Wire Line
-	7050 3850 7050 3800
-Wire Wire Line
-	7650 4150 7650 4100
 Wire Wire Line
 	7000 3600 7050 3600
@@
 F 3 "~" H 7650 5600 50  0001 C CNN
 	1    7650 5600
-	0    1    1    0
+	0    -1   1    0
 $EndComp
 Wire Wire Line
@@
 P 3000 3800
 F 0 "AE1" H 3144 3839 50  0000 L CNN
-F 1 "SGGP.12A" H 3144 3748 50  0000 L CNN
-F 2 "Connector_Coaxial:U.FL_Molex_MCRF_73412-0110_Vertical" H 3000 3900 50  0001 C CNN
+F 1 "U.FL" H 3144 3748 50  0000 L CNN
+F 2 "Connector_Coaxial:U.FL_Hirose_U.FL-R-SMT-1_Vertical" H 3000 3900 50  0001 C CNN
 F 3 "~" H 3000 3900 50  0001 C CNN
 	1    3000 3800
@@
 Wire Wire Line
 	950  1400 500  1400
-Wire Wire Line
-	6100 5200 5750 5200
 Text Label 6100 5200 2    50   ~ 0
 3v3
 Wire Wire Line
 	5650 5300 5750 5300
-Wire Wire Line
-	5750 5300 5750 5200
-Connection ~ 5750 5200
-Wire Wire Line
-	5750 5200 5650 5200
 Wire Wire Line
 	6100 5400 5650 5400
@@
 Wire Wire Line
 	5450 4850 5750 4850
-Wire Wire Line
-	5750 4850 5750 5200
 $Comp
 L Device:C_Small C7
@@
 $EndComp
 $Comp
-L power:GNDA #PWR0114
-U 1 1 6192ABB2
-P 7650 4150
-F 0 "#PWR0114" H 7650 3900 50  0001 C CNN
-F 1 "GNDA" H 7655 3977 50  0000 C CNN
-F 2 "" H 7650 4150 50  0001 C CNN
-F 3 "" H 7650 4150 50  0001 C CNN
-	1    7650 4150
-	1    0    0    -1
-$EndComp
-$Comp
 L power:GNDA #PWR0115
 U 1 1 6192FCED
@@
 Text Label 9400 4500 2    50   ~ 0
 3V3
-Wire Wire Line
-	1950 2150 1850 2150
 $Comp
 L Sensor_Motion:ADXL343 U12
@@
 P 10300 3450
 F 0 "U12" H 10844 3496 50  0000 L CNN
-F 1 "ADXL343" H 10844 3405 50  0000 L CNN
+F 1 "ADXL375" H 10844 3405 50  0000 L CNN
 F 2 "Package_LGA:LGA-14_3x5mm_P0.8mm_LayoutBorder1x6y" H 10300 3450 50  0001 C CNN
 F 3 "https://www.analog.com/media/en/technical-documentation/data-sheets/ADXL343.pdf" H 10300 3450 50  0001 C CNN
@@
 $EndComp
 Wire Wire Line
-	5350 3500 4850 3500
-Text Label 4850 3500 0    50   ~ 0
+	5350 3700 4850 3700
+Text Label 4850 3700 0    50   ~ 0
 LED_B
 Wire Wire Line
@@
 LED_R
 Wire Wire Line
-	5350 3700 4850 3700
-Text Label 4850 3700 0    50   ~ 0
+	5350 3500 4850 3500
+Text Label 4850 3500 0    50   ~ 0
 LED_G
 $Comp
@@
 	4650 2400 4600 2400
 Wire Wire Line
-	4950 2500 5350 2500
-Text Label 4950 2600 0    50   ~ 0
-EXT_RX
-Text Label 4950 2500 0    50   ~ 0
-EXT_TX
-Wire Wire Line
 	4750 1700 5350 1700
 Connection ~ 4600 2400
-Wire Wire Line
-	5350 2600 4950 2600
 Connection ~ 7050 3450
 Wire Wire Line
 	7050 3450 7050 3400
-Wire Wire Line
-	7650 3850 7650 4000
-Wire Wire Line
-	7050 3850 7650 3850
-Wire Wire Line
-	7650 4000 7650 4100
-Connection ~ 7650 4000
-Connection ~ 7650 4100
-Wire Wire Line
-	7000 4100 7650 4100
 Wire Wire Line
 	7000 3700 7350 3700
@@
 Wire Wire Line
 	5600 7200 5400 7200
-$Comp
-L Connector_Generic:Conn_01x04 J5
-U 1 1 6290413B
-P 8400 3150
-F 0 "J5" H 8318 2725 50  0000 C CNN
-F 1 "SWD port" H 8318 2816 50  0000 C CNN
-F 2 "Connector_PinHeader_1.27mm:PinHeader_1x04_P1.27mm_Vertical" H 8400 3150 50  0001 C CNN
-F 3 "~" H 8400 3150 50  0001 C CNN
-	1    8400 3150
-	-1   0    0    1
-$EndComp
-Wire Wire Line
-	8600 3250 8700 3250
-Wire Wire Line
-	8700 3250 8700 3300
-Wire Wire Line
-	8600 3150 8950 3150
-Wire Wire Line
-	8950 3050 8600 3050
+Wire Wire Line
+	8750 3250 8750 3300
+Wire Wire Line
+	8600 3100 8950 3100
 Wire Wire Line
 	8950 2950 8600 2950
+Wire Wire Line
+	8950 2800 8600 2800
+Text Label 8950 2800 2    50   ~ 0
+3V3
 Text Label 8950 2950 2    50   ~ 0
-3V3
-Text Label 8950 3050 2    50   ~ 0
 SWDIO
-Text Label 8950 3150 2    50   ~ 0
+Text Label 8950 3100 2    50   ~ 0
 SWCLK
 $Comp
 L power:GND #PWR0126
 U 1 1 62954B0E
-P 8700 3300
-F 0 "#PWR0126" H 8700 3050 50  0001 C CNN
-F 1 "GND" H 8705 3127 50  0000 C CNN
-F 2 "" H 8700 3300 50  0001 C CNN
-F 3 "" H 8700 3300 50  0001 C CNN
-	1    8700 3300
+P 8750 3300
+F 0 "#PWR0126" H 8750 3050 50  0001 C CNN
+F 1 "GND" H 8755 3127 50  0000 C CNN
+F 2 "" H 8750 3300 50  0001 C CNN
+F 3 "" H 8750 3300 50  0001 C CNN
+	1    8750 3300
 	1    0    0    -1
 $EndComp
@@
 3V3_BAK
 Connection ~ 2400 950
-Connection ~ 1850 2150
-Wire Wire Line
-	1850 3000 1850 2150
 Text Notes 2850 1300 0    50   ~ 0
 no cap according to datasheet\nbuilt in reverse voltage\n
@@
 Text Label 2050 4450 0    50   ~ 0
 3V3
-Connection ~ 3250 4450
-Text Label 3450 4450 2    50   ~ 0
-3V3
-Wire Wire Line
-	3250 4450 3450 4450
 Wire Wire Line
 	3100 4450 3250 4450
@@
 Wire Wire Line
 	5350 2000 4900 2000
-Wire Wire Line
-	3250 4900 3250 4800
-Connection ~ 3250 4800
 $Comp
 L Device:D_Schottky_Small D3
@@
 Wire Wire Line
 	1400 1700 1400 2150
-Wire Wire Line
-	1400 2150 1850 2150
-Text Notes 3350 -450 0    394  ~ 0
-UFL VERSION
-Text Notes 4500 4400 1    394  ~ 0
-UFL VERSION
+$Comp
+L Device:Antenna AE2
+U 1 1 6124D6BA
+P 7850 3600
+F 0 "AE2" H 7930 3589 50  0000 L CNN
+F 1 "ANT-868-PW-LP" H 7930 3498 50  0000 L CNN
+F 2 "custom:ANT-868-PW-LP" H 7850 3600 50  0001 C CNN
+F 3 "~" H 7850 3600 50  0001 C CNN
+	1    7850 3600
+	1    0    0    -1
+$EndComp
+Wire Wire Line
+	7050 3800 7050 3850
+$Comp
+L power:GNDA #PWR0114
+U 1 1 612A28B4
+P 7150 4150
+F 0 "#PWR0114" H 7150 3900 50  0001 C CNN
+F 1 "GNDA" H 7155 3977 50  0000 C CNN
+F 2 "" H 7150 4150 50  0001 C CNN
+F 3 "" H 7150 4150 50  0001 C CNN
+	1    7150 4150
+	1    0    0    -1
+$EndComp
+Wire Wire Line
+	7000 4100 7150 4100
+Wire Wire Line
+	7150 4100 7150 4150
+Wire Wire Line
+	7050 3850 7150 3850
+Wire Wire Line
+	7150 3850 7150 4100
+Connection ~ 7050 3850
+Wire Wire Line
+	7050 3850 7050 3900
+Connection ~ 7150 4100
+Wire Wire Line
+	7000 4000 7850 4000
+Wire Wire Line
+	7850 4000 7850 3800
+Wire Wire Line
+	1400 2150 1950 2150
+Connection ~ 3250 4800
+Wire Wire Line
+	3250 4900 3250 4800
+Wire Wire Line
+	3450 4450 3250 4450
+Connection ~ 3250 4450
+Text Label 3450 4450 2    50   ~ 0
+3V3
+Wire Wire Line
+	5650 5200 5750 5200
+Wire Wire Line
+	5750 5300 5750 5200
+Connection ~ 5750 5200
+Wire Wire Line
+	5750 4850 5750 5200
+Wire Wire Line
+	6300 5200 6300 5300
+Wire Wire Line
+	5750 5200 6300 5200
+$Comp
+L Device:C_Small C4
+U 1 1 61501811
+P 6300 5400
+F 0 "C4" H 6392 5446 50  0000 L CNN
+F 1 "0.1u" H 6392 5355 50  0000 L CNN
+F 2 "Capacitor_SMD:C_0603_1608Metric_Pad1.08x0.95mm_HandSolder" H 6300 5400 50  0001 C CNN
+F 3 "~" H 6300 5400 50  0001 C CNN
+	1    6300 5400
+	1    0    0    -1
+$EndComp
+Wire Wire Line
+	6300 5500 6300 5550
+$Comp
+L power:GND #PWR0129
+U 1 1 6152CE8D
+P 6300 5550
+F 0 "#PWR0129" H 6300 5300 50  0001 C CNN
+F 1 "GND" H 6305 5377 50  0000 C CNN
+F 2 "" H 6300 5550 50  0001 C CNN
+F 3 "" H 6300 5550 50  0001 C CNN
+	1    6300 5550
+	1    0    0    -1
+$EndComp
+$Comp
+L Connector_Generic:Conn_01x01 J3
+U 1 1 61596691
+P 8400 3250
+F 0 "J3" H 8800 3250 50  0000 C CNN
+F 1 "GND" H 8550 3250 50  0000 C CNN
+F 2 "custom:just_a_pad" H 8400 3250 50  0001 C CNN
+F 3 "~" H 8400 3250 50  0001 C CNN
+	1    8400 3250
+	-1   0    0    1
+$EndComp
+$Comp
+L Connector_Generic:Conn_01x01 J7
+U 1 1 615F2DA2
+P 8400 3100
+F 0 "J7" H 8800 3100 50  0000 C CNN
+F 1 "SWCLK" H 8600 3100 50  0000 C CNN
+F 2 "custom:just_a_pad" H 8400 3100 50  0001 C CNN
+F 3 "~" H 8400 3100 50  0001 C CNN
+	1    8400 3100
+	-1   0    0    1
+$EndComp
+Wire Wire Line
+	8600 3250 8750 3250
+$Comp
+L Connector_Generic:Conn_01x01 J6
+U 1 1 61608EF1
+P 8400 2950
+F 0 "J6" H 8800 2950 50  0000 C CNN
+F 1 "SWDIO" H 8600 2950 50  0000 C CNN
+F 2 "custom:just_a_pad" H 8400 2950 50  0001 C CNN
+F 3 "~" H 8400 2950 50  0001 C CNN
+	1    8400 2950
+	-1   0    0    1
+$EndComp
+$Comp
+L Connector_Generic:Conn_01x01 J5
+U 1 1 61609152
+P 8400 2800
+F 0 "J5" H 8800 2800 50  0000 C CNN
+F 1 "3V3" H 8550 2800 50  0000 C CNN
+F 2 "custom:just_a_pad" H 8400 2800 50  0001 C CNN
+F 3 "~" H 8400 2800 50  0001 C CNN
+	1    8400 2800
+	-1   0    0    1
+$EndComp
+Wire Wire Line
+	5350 2600 4950 2600
+Text Label 4950 2500 0    50   ~ 0
+EXT_TX
+Text Label 4950 2600 0    50   ~ 0
+EXT_RX
+Wire Wire Line
+	4950 2500 5350 2500
 $EndSCHEMATC
