File: electronics/mini_controller4/mini_controller.kicad_pcb (KiCad board)
At the start: 4 copper layers, 13 x 53.6 mm, 48 parts, among them J1 Conn_01x06, J2 Conn_01x05, J3 GND, J5 3V3, J6 SWDIO, J7 SWCLK, Q1 MMBT3904, U1 JST-RCY, U10 SKY65723-81, U2 BU33SD5WG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

Commit message: routing finished v4
Parts:
- removed J3: GND, custom:just_a_pad
- removed J5: 3V3, custom:just_a_pad
- H1, H2: value MountingHole -> MountingHole_Pad; footprint MountingHole:MountingHole_2.2mm_M2_ISO7380 -> MountingHole:MountingHole_2.2mm_M2_ISO7380_Pad_TopOnly; moved to B.Cu
- J2: value Conn_01x05 -> Conn_01x06; footprint Connector_JST:JST_SH_BM05B-SRSS-TB_1x05-1MP_P1.00mm_Vertical -> Connector_JST:JST_SH_BM06B-SRSS-TB_1x06-1MP_P1.00mm_Vertical
- J6, J7: moved to B.Cu
- moved J6 61.4 mm to (193.8, 95.5)
- moved J7 42.1 mm to (181.6, 95.5)
- moved H1 9.65 mm to (192.5, 78.7)
- moved H2 9.65 mm to (182.8, 78.7)
- moved U10 1.92 mm to (184.9, 102.1)
- moved C6 1.84 mm to (183.0, 103.6), turned to 0 degrees
- moved R13 1.27 mm to (182.6, 113.5)
- moved R15 1.27 mm to (182.6, 112.3)
- moved R19 1.27 mm to (184.9, 113.5)
- moved C1 1.27 mm to (187.8, 112.0), turned to 90 degrees
- moved R20 1.27 mm to (184.9, 112.3)
- moved R17 0.92 mm to (184.5, 121.5)
- moved R16 0.92 mm to (183.1, 123.7)
- moved R18 0.91 mm to (183.1, 121.5)
- moved R14 0.91 mm to (184.5, 123.7)
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Connections:
- H1 pad 1: (no net) -> GND
- H2 pad 1: (no net) -> GND
- J2 pad 1: GND -> /EXT_MISC
- J2 pad 2: /EXT_RX -> /BOOT0
- J2 pad 3: /EXT_TX -> /3V3
- J2 pad 4: /3V3 -> /EXT_TX
- J2 pad 5: /BOOT0 -> /EXT_RX
- U3 pad 11: (no net) -> GND
- U3 pad 12: (no net) -> GND
- U3 pad 13: (no net) -> /SDA3
- U3 pad 14: (no net) -> /SCL3
- U3 pad 2: Net-(U3-Pad2) -> GND
- U3 pad 3: (no net) -> /3V3
- U3 pad 4: Net-(U3-Pad2) -> GND
- U3 pad 5: Net-(U3-Pad2) -> GND
- U3 pad 7: (no net) -> /3V3
- U7 pad 1: (no net) -> /FLASH_CS
- U7 pad 2: (no net) -> /FLASH_MISO
- U7 pad 3: (no net) -> /3V3
- U7 pad 4: (no net) -> GND
- U7 pad 5: (no net) -> /FLASH_MOSI
- U7 pad 6: (no net) -> /FLASH_SCK
- U7 pad 7: (no net) -> /3V3
- U8 pad 13: /PYRO_4_EN -> (no net)
- U8 pad 16: /EXT_TX -> (no net)
- U8 pad 17: /EXT_RX -> (no net)
- U8 pad 18: (no net) -> /FLASH_CS
- U8 pad 19: (no net) -> /FLASH_SCK
- U8 pad 20: (no net) -> /FLASH_MISO
- U8 pad 21: (no net) -> /FLASH_MOSI
- U8 pad 24: /PYRO_3_EN -> (no net)
- U8 pad 25: /PYRO_1_EN -> (no net)
- U8 pad 46: (no net) -> /EXT_RX
- U8 pad 47: (no net) -> /EXT_TX
- U8 pad 54: (no net) -> /EXT_MISC
- U8 pad 55: (no net) -> /PYRO_4_EN
- U8 pad 56: (no net) -> /PYRO_3_EN
- U8 pad 57: (no net) -> /PYRO_2_EN
- U8 pad 58: (no net) -> /PYRO_1_EN
- U8 pad 7: /PYRO_2_EN -> (no net)
Routing:
- net /3V3: track 0.00 -> 99.4 mm, vias 0 -> 6
- net GND: track 0.00 -> 77.6 mm, vias 0 -> 17
- net /PYRO_4_EN: track 0.00 -> 36.8 mm, vias 0 -> 2
- net /SDA3: track 0.00 -> 31.8 mm, vias 0 -> 2
- net /SCL3: track 0.00 -> 31.7 mm, vias 0 -> 2
- net /BAT_SENSE: track 0.00 -> 31.5 mm, vias 0 -> 2
- net /PYRO_3_EN: track 0.00 -> 31.3 mm, vias 0 -> 2
- net /LED: track 0.00 -> 27.5 mm, vias 0 -> 2
- net /GPS_TX: track 0.00 -> 25.0 mm, vias 0 -> 2
- net /GPS_RX: track 0.00 -> 24.8 mm, vias 0 -> 2
- net /SWDIO: track 0.00 -> 22.3 mm, vias 0 -> 1
- net /PYRO_1_EN: track 0.00 -> 21.9 mm, vias 0 -> 2
- net /SWCLK: track 0.00 -> 21.0 mm, vias 0 -> 2
- net /PYRO_2_EN: track 0.00 -> 19.4 mm, vias 0 -> 2
- net /FLASH_CS: track 0.00 -> 17.1 mm, vias 0 -> 1
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- added copper zone on B.Cu, net GND
- added copper zone on F.Cu, net GND
- added copper zone on In1.Cu, net GND
- added copper zone on In2.Cu, net GND
Other:
- board text added: "+"
- board text added: "1"
- board text added: "2"
- board text added: "3"
- board text added: "4"

Commit message: misc
Other:
- outline, holes or cut-outs redrawn
