File: electronics/mini_controller4/mini_controller.sch (KiCad schematic (older format))
At the start: 48 parts, among them J1 Conn_01x06, J2 Conn_01x05, J3 GND, J5 3V3, J6 SWDIO, J7 SWCLK, Q1 MMBT3904, U1 JST-RCY, U10 SKY65723-81, U2 BU33SD5WG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

Commit message: routing finished v4
Parts:
- removed H1, H2: MountingHole, MountingHole:MountingHole_2.2mm_M2_ISO7380, symbol Mechanical:MountingHole
- removed J2: Conn_01x05, Connector_JST:JST_SH_BM05B-SRSS-TB_1x05-1MP_P1.00mm_Vertical, symbol Connector_Generic:Conn_01x05
- removed J3: GND, custom:just_a_pad, symbol Connector_Generic:Conn_01x01
- removed J5: 3V3, custom:just_a_pad, symbol Connector_Generic:Conn_01x01
- added H1, H2: MountingHole_Pad, MountingHole:MountingHole_2.2mm_M2_ISO7380_Pad_TopOnly, symbol Mechanical:MountingHole_Pad
- added J2: Conn_01x06, Connector_JST:JST_SH_BM06B-SRSS-TB_1x06-1MP_P1.00mm_Vertical, symbol Connector_Generic:Conn_01x06
Connections:
- net 3V3: now also U3.3 (RES), U3.7 (~CS), U7.3 (~WP~/IO2), U7.7 (~HOLD~/IO3), J2.3 (Pin_3)
- net BOOT0: now also J2.2 (Pin_2)
- net EXT_RX: now also U8.46 (PA10_USART1_RX), J2.5 (Pin_5); no longer U8.17 (PA3_RXD_A)
- net EXT_TX: now also U8.47 (PA9_USART1_TX), J2.4 (Pin_4); no longer U8.16 (PA2_TXD_A)
- net FLASH_CS: now also U7.1 (~CS)
- net FLASH_MISO: now also U7.2 (SO/IO1)
- net FLASH_MOSI: now also U7.5 (SI/IO0)
- net FLASH_SCK: now also U7.6 (SCK)
- net GND: now also U3.11 (RES), U3.12 (SDO/ADDR), U3.2 (GND), U3.4 (GND), U3.5 (GND), U7.4 (GND), H1.1, H2.1, J2.6 (Pin_6)
- net PYRO_1_EN: now also U8.58 (PB7_SDA); no longer U8.25 (PB1_IO_INT2)
- net PYRO_2_EN: now also U8.57 (PB6_SCL); no longer U8.7 (PC3)
- net PYRO_3_EN: now also U8.56 (PB5); no longer U8.24 (PB0_IO_INT1)
- net PYRO_4_EN: now also U8.55 (PD2); no longer U8.13 (PA0)
- net SCL3: now also U3.14 (SCL/SCLK)
- net SDA3: now also U3.13 (SDA/SDI/SDIO)
- net EXT_MISC: now reaches U8.54 (PC12)
- net EXT_MISC: now also J2.1 (Pin_1)
- net 3V3_BAK: no longer names the net of U4.6 (V_BCKP)
Other:
- moved on the sheet: C4, U3

Commit message: misc
Parts:
- D1, D3: value ZLLS350TA -> XBS053V15R-G
- D2: value LED -> APHHS1005CGCK
- R1: value 400 -> 500
Other:
- note added: "Accelerometer"
- note added: "SWD"
- moved on the sheet: C1, C4, C7, J6, J7, U3, U7, U9
